Commit message: fix package name

File: realsense2_description/urdf/_d415.urdf.xacro (robot description, xacro)
@@ -46,5 +46,5 @@
         <geometry>
           <!-- <box size="${d415_cam_width} ${d415_cam_height} ${d415_cam_depth}"/> -->
-	         <mesh filename="package://realsense2_description/meshes/d415.stl" />
+	         <mesh filename="package://realsense2_description_pal_robotics_forked/meshes/d415.stl" />
         </geometry>
         <material name="${name}_aluminum"/>

File: realsense2_description/urdf/_d435.urdf.xacro (robot description, xacro)
@@ -48,6 +48,6 @@
         <geometry>
           <!-- <box size="${d435_cam_width} ${d435_cam_height} ${d435_cam_depth}"/> -->
-          <mesh filename="package://realsense2_description/meshes/d435.dae" />
-          <!--<mesh filename="package://realsense2_description/meshes/d435/d435.dae" />-->
+          <mesh filename="package://realsense2_description_pal_robotics_forked/meshes/d435.dae" />
+          <!--<mesh filename="package://realsense2_description_pal_robotics_forked/meshes/d435/d435.dae" />-->
         </geometry>
         <material name="${name}_aluminum"/>

File: realsense2_description/urdf/_r410.urdf.xacro (robot description, xacro)
@@ -39,5 +39,5 @@
         <geometry>
           <box size="${r410_cam_width} ${r410_cam_height} ${r410_cam_depth}"/>
-          <!--<mesh filename="package://realsense2_description/meshes/r410/r410.dae" />-->
+          <!--<mesh filename="package://realsense2_description_pal_robotics_forked/meshes/r410/r410.dae" />-->
         </geometry>
         <material name="${name}_aluminum"/>

File: realsense2_description/urdf/_r430.urdf.xacro (robot description, xacro)
@@ -40,5 +40,5 @@
         <geometry>
           <box size="${r430_cam_width} ${r430_cam_height} ${r430_cam_depth}"/>
-          <!--<mesh filename="package://realsense2_description/meshes/r430/r430.dae" />-->
+          <!--<mesh filename="package://realsense2_description_pal_robotics_forked/meshes/r430/r430.dae" />-->
         </geometry>
         <material name="${name}_aluminum"/>

File: realsense2_description/urdf/_t265.urdf.xacro (robot description, xacro)
@@ -38,5 +38,5 @@
       <origin xyz="0 0 0" rpy="0 0 0"/>
         <geometry>
-            <mesh filename="package://realsense2_description/meshes/t265.stl" />
+            <mesh filename="package://realsense2_description_pal_robotics_forked/meshes/t265.stl" />
         </geometry>
         <material name="${name}_aluminum"/>
@@ -45,5 +45,5 @@
         <origin xyz="0 0 0" rpy="0 0 0"/>
         <geometry>
-          <mesh filename="package://realsense2_description/meshes/t265.stl" />
+          <mesh filename="package://realsense2_description_pal_robotics_forked/meshes/t265.stl" />
         </geometry>
       </collision>
